File: design-files/c64-rom-326298.kicad_sch (KiCad schematic)
At the start: 16 parts, among them J1 Conn_01x12_Pin, J2 Conn_01x12_Pin, J3 Conn_01x02_Pin, J4 Conn_01x04_Pin, J5 Conn_01x12_Pin, SW101 SW_DIP_x02, SW102 SW_DIP_x02, SW103 SW_DIP_x02, U101 SST39SF010, U102 GAL22V10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

Commit message: Fix name / company on schematic sheet.
Other:
- company: Jason R. Thorpe -> Copyright (c) 2023 Jason R. Thorpe. See LICENSE.
- title: C64-ROM-326298 -> Commodore 64 326298 ROM Replacer / Selector
Changed lines of the file:
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@@
   (paper "A4")
   (title_block
-    (title "C64-ROM-326298")
+    (title "Commodore 64 326298 ROM Replacer / Selector")
     (date "2023-10-28")
     (rev "1.0")
-    (company "Jason R. Thorpe")
+    (company "Copyright (c) 2023 Jason R. Thorpe. See LICENSE.")
   )
   (junction (at 179.959 99.06) (diameter 0) (color 0 0 0 0)
